Commit message: feat(description): A6 evidence checks, config id and verify_a6.sh
Add the S5 verification for openamrobot_upperbody_description (part of #7):

- T02: check_urdf on the 12 T01 expansions plus openarm on gazebo and real
  at mast_1350, and the planar-flag expansions (extra, labelled). A missing
  check_urdf is a FAIL, not a skip.
- T07/T08: every link with an inertial or visual has a collision or is
  collision_free with a reason (FAIL); collision mesh == visual mesh is
  listed (WARN only).
- T09: mass > 0, Ixx/Iyy/Izz > 0, principal moments > 0, triangle
  inequality, tensor positive-definite (numpy eigenvalues).
- T10: modelled mass by owner (base, mast, openarm_*, sensors), the not
  modelled list in words, the W01 line; FAIL only above gross_mass_limit.
- E01: approximate assembled height (zero pose, frame origins and
  box/cylinder/sphere extents, no mesh extents) against max_assembled_height;
  WARN for analysis mast IDs, FAIL for the release one.
- W02 (WARN): KDL converts base_planar_joint to a fixed joint. Observed from
  a real robot_state_publisher; recorded as a consumer limitation that does
  not affect A6 acceptance. Planar base motion for A7 comes from Gazebo's
  odom -> base_link, never from robot_state_publisher.
- scripts/print_config_id.py: full sha256:<64 hex> over the canonical
  expanded URDF, mast_id, arm_package, hardware_profile, datums.revision and
  the pinned openarm_description commit. C01 asserts the format and
  validates it against the pattern in the installed C9 schema (SKIP with the
  reason if openamrobot-interfaces is not in the workspace).
- Evidence directory: default is now <workspace>/evidence, found from the
  package share path; OPENAMR_EVIDENCE_DIR overrides; never a temp dir (T04's
  sidecar moves with it).
- T13: visualization constants (DATUMS.md) must be visual-only, a named
  property with a comment saying so, and are listed in the evidence. The
  comment on openamr_sensor_marker_edge now says it; the expansion is
  unchanged.
- scripts/verify_a6.sh runs colcon test, the T02 matrix, datums_report.py
  and the config ids, and writes evidence/<UTC ts>_dev.json
  (evidence_class static+mock). Exit status is non-zero iff any check is FAIL.
  T14-T16 and L01 are SKIP (S7), not passed.

Assisted-by: Claude Code
Signed-off-by: Tushar Goel <Slash8860300674@gmail.com>

File: ros2/src/openamrobot_upperbody_description/urdf/upper_sensors.xacro (robot description, xacro)
@@ -13,6 +13,7 @@
 -->
 <robot xmlns:xacro="http://www.ros.org/wiki/xacro">
-  <!-- Marker box edge, metres. A drawing aid like the 1/2 and 1/12 of a cuboid inertia, not a hardware dimension: no
-       collision, no inertial and no datum depends on it. -->
+  <!-- Visualization constant (DATUMS.md): edge, in metres, of the marker box drawn for each camera frame. It describes
+       how the model is drawn, not the robot, so it is not a datum. It may appear only inside a <visual>: no collision,
+       no inertial, no joint origin and no datum depends on it (T13 enforces this). -->
   <xacro:property name="openamr_sensor_marker_edge" value="0.04"/>
   <xacro:macro name="openamr_camera_frames" params="name parent pose">
