Commit message: test(description): the finger-mimic multiplier is read from upstream's yaml, and a hard-coded one is caught
P06 disclosed that replacing the multiplier with a literal was not caught, and called it harmless because upstream
only uses it inside a commented-out joint. That stops being true once Gazebo computes with it.

The property moves from inside the mock/real branch to file scope in ros2_control.xacro so a probe file can read it
(a macro-local property was invisible, and xacro does not evaluate comments, so no expansion showed it). The expansion
of mock, gazebo and real is byte-identical before and after.

test_t15_finger_mimic_multiplier.py checks the value against an independent read of joint_mimics.yaml and the source
expression for a load_yaml call, so a wrong number and a literal equal to today's value are both caught. Demonstrated on
mutated copies, and on the real file: hard-coding 1.0 and -1.0 fail it.

Assisted-by: Claude Code
Signed-off-by: Tushar Goel <Slash8860300674@gmail.com>

File: ros2/src/openamrobot_upperbody_description/urdf/ros2_control.xacro (robot description, xacro)
@@ -16,4 +16,11 @@
 <robot xmlns:xacro="http://www.ros.org/wiki/xacro">
   <xacro:include filename="$(find openarm_description)/assets/robot/openarm_v2.0/urdf/ros2_control/openarm.bimanual.ros2_control.xacro"/>
+  <!-- The finger-mimic multiplier is READ from upstream's joint_mimics.yaml, never written in here (the same expression
+       upstream's openarm_v20.urdf.xacro uses). File scope, not inside a macro, so every profile sees one value and
+       test_t15_finger_mimic_multiplier.py can read it: in mock and real upstream only uses it in a commented-out joint,
+       so nothing in an expansion would otherwise show a hard-coded replacement. -->
+  <xacro:property name="pinch_mimics_file" value="$(find openarm_description)/assets/end_effector/pinch_gripper/config/joint/joint_mimics.yaml"/>
+  <xacro:property name="pinch_mimics_dict" value="${xacro.load_yaml(pinch_mimics_file)}"/>
+  <xacro:property name="pinch_finger_mimic_multiplier" value="${pinch_mimics_dict['joint2']['multiplier'] if 'joint2' in pinch_mimics_dict else 1.0}"/>
   <!-- One joint with the interfaces the upstream macro declares (openarm.bimanual.ros2_control.xacro,
        configure_joint): position, velocity and effort commands; position, velocity and effort state, all starting at 0.
@@ -42,7 +49,4 @@
       <xacro:property name="gains_file" value="${openarm_robot_root + '/config/arm/control/control_gains.yaml'}"/>
       <xacro:property name="gains_dict" value="${xacro.load_yaml(gains_file)}"/>
-      <xacro:property name="pinch_mimics_file" value="$(find openarm_description)/assets/end_effector/pinch_gripper/config/joint/joint_mimics.yaml"/>
-      <xacro:property name="pinch_mimics_dict" value="${xacro.load_yaml(pinch_mimics_file)}"/>
-      <xacro:property name="pinch_finger_mimic_multiplier" value="${pinch_mimics_dict['joint2']['multiplier'] if 'joint2' in pinch_mimics_dict else 1.0}"/>
       <xacro:openarm_bimanual_ros2_control
         arm_type="v20"

Commit message: feat(description): the gazebo profile loads gz_ros2_control into the model with the arm controller yaml
Adds the Gazebo-side half of ADR-003 to the gazebo branch of ros2_control.xacro: a model plugin,
filename gz_ros2_control-system, class gz_ros2_control::GazeboSimROS2ControlPlugin, whose <parameters> is
openamrobot_upperbody_control's arm_controllers.yaml by installed path ($(find ...)), the one controller file every
profile uses. mock and real expand exactly as before.

Names read from the installed Jazzy gz_ros2_control 1.2.20, not from documentation: libgz_ros2_control-system.so
registers the class, libgz_hardware_plugins.so registers gz_ros2_control/GazeboSimSystem. The library also refuses to
load anywhere but a model ("is not a model. Please make sure that Gazebo ROS 2 Control is attached to a valid model"),
which is why this is a model plugin carried by the description and the world file holds only world systems.

finger_joint2 stays out of ros2_control, replacing P06's TODO with what was measured: Jazzy's ros2_control rejects upstream's
commented-out block ("Activated mimic joints cannot have command interfaces"), and the URDF <mimic> is honoured by the
Bullet-Featherstone physics engine on its own. The package.xml does not depend on openamrobot_upperbody_control for the
$(find): control already test_depends on this package, so a dependency back is a cycle.

T15 gains tests for the plugin (model plugin, installed yaml path, absent in mock and real, platform-sw's DiffDrive plugin
untouched) and one that reads the plugin names out of the installed library.

Assisted-by: Claude Code
Signed-off-by: Tushar Goel <Slash8860300674@gmail.com>

File: ros2/src/openamrobot_upperbody_description/urdf/ros2_control.xacro (robot description, xacro)
@@ -60,11 +60,31 @@
     </xacro:if>
     <xacro:if value="${hardware_profile == 'gazebo'}">
+      <!-- The Gazebo side of gz_ros2_control: a MODEL plugin that loads a controller manager next to the model and
+           hands it the controller parameters. A model plugin and not a world plugin: the library refuses anything else
+           ("is not a model. Please make sure that Gazebo ROS 2 Control is attached to a valid model"). A <gazebo> element
+           with no reference becomes a plugin of the model when ros_gz_sim converts the URDF to SDF. Filename and class were
+           read from the installed Jazzy gz_ros2_control 1.2.20, not from documentation: libgz_ros2_control-system.so
+           registers gz_ros2_control::GazeboSimROS2ControlPlugin (libgz_hardware_plugins.so registers GazeboSimSystem).
+           The controllers are the same file every profile uses (ADR-003). The world, physics, sensors and the launch that
+           spawns this model are simulation bringup and live in openamrobot_upperbody_gazebo. -->
+      <gazebo>
+        <plugin filename="gz_ros2_control-system" name="gz_ros2_control::GazeboSimROS2ControlPlugin">
+          <parameters>$(find openamrobot_upperbody_control)/config/arm_controllers.yaml</parameters>
+        </plugin>
+      </gazebo>
       <ros2_control name="openamr_arms_gazebo" type="system">
         <hardware>
           <plugin>gz_ros2_control/GazeboSimSystem</plugin>
         </hardware>
-        <!-- openarm_{left,right}_finger_joint2 is left out as upstream leaves it out of ros2_control.
-             TODO(gazebo, A7): whether gz_ros2_control then follows the URDF <mimic> on its own, or needs
-             <param name="mimic"> here, is unverified: nothing launches Gazebo in P06. -->
+        <!-- openarm_{left,right}_finger_joint2 is left out, as upstream leaves it out of ros2_control (decided P09, measured
+             in Gazebo Harmonic 8.15 with gz_ros2_control 1.2.20):
+               - the URDF <mimic> becomes an SDF mimic constraint, which the Bullet-Featherstone engine honours and the
+                 default DART engine does not ("chosen physics engine does not support mimic constraints"). With
+                 Bullet-Featherstone finger_joint2 follows finger_joint1 on its own; openamrobot_upperbody_gazebo selects it.
+               - declaring finger_joint2 here the way upstream's commented-out block does cannot load: this ros2_control
+                 refuses "Activated mimic joints cannot have command interfaces", and with <param name="mimic"> and no
+                 command interface it adds nothing the physics does not already do.
+             So nothing is declared for it. The multiplier it follows is the URDF's own, from the same yaml as
+             pinch_finger_mimic_multiplier above. -->
         <xacro:openamr_gazebo_arm_joint joint_name="openarm_left_joint1"/>
         <xacro:openamr_gazebo_arm_joint joint_name="openarm_left_joint2"/>
