Commit message: feat(description,moveit,bringup): lift column placeholder boxes, M07 WARN at upstream limits, re-derived ACM
Follow-ups (a) and (b) to 49d2368, accepted by Alex on 16 Oct.

(a) The lift column gets placeholder geometry: a 240 x 240 mm box (datum
lift_column_section, placeholder) on both stages, visual and collision,
named placeholder_lift_column_*: the fixed stage on lift_column_base_link
(retracted length) and the moving stage on lift_carriage_link (stroke,
below the carriage). It is an opt-in macro parameter, column_geometry
(default none, as on main); combined_robot.xacro passes the section.
frame_contract.yaml no longer calls lift_column_base_link collision-free.

The collision matrix is re-derived with regenerate_acm.sh --write: 95
pairs (20 upstream + 17 Adjacent + 58 ConstantTransform), was 83; 535 of
630 pairs enabled, was 478. The SRDF, acm_generation.yaml, the count
assertions of test_acm_derive.py and test_m03_acm_sampling.py, the
MoveIt README and the CHANGELOG follow.

(b) M07 reports WARN, not FAIL, for openarm_{left,right}_finger_joint1
and openarm_{left,right}_joint4, reason "rest pose at an upstream limit",
when they rest within the margin on either side of that limit. Any other
joint within the margin, or one of those further past its limit than the
margin, is still a FAIL.

Co-Authored-By: Claude Opus 5.5 <noreply@anthropic.com>
Claude-Session: https://claude.ai/code/session_01RtnAs3hZ9W2iEfaMcCvWng
Signed-off-by: Alex Reznichenko <info@botshare.ai>

File: ros2/src/openamrobot_upperbody_description/urdf/combined_robot.xacro (robot description, xacro)
@@ -90,5 +90,6 @@
        Shape: a uniform box of the column's section (datum, axis convention x fore-aft, y lateral) and its retracted length (option B's
        config), centred at half of that length above lift_column_base_link. All of the mass is on the fixed side (the catalogue
-       does not split it). No collision and no visual: the column body's lateral extent is not sourced. -->
+       does not split it). Visual and collision: placeholder boxes of the same section on both stages (column_geometry), until the
+       supplier drawing; the column body's lateral extent is not sourced. -->
   <xacro:property name="lift_mass_by_column" lazy_eval="false"
                   value="${dict(dold_v4_350=dt['lift_mass_dold_v4_350']['value'], tl3_400=dt['lift_mass_tl3_400']['value'])}"/>
@@ -112,5 +113,6 @@
   <xacro:openamrobot_upperbody parent="base_footprint" column="${column}" base_plate="${base_plate}" head_pitch="${head_pitch}"
                                base_tilt="${base_tilt}" column_axis_x_bp000="${dt['column_axis_x_bp000']['value']}"
-                               emit_arm_mounts="${arm_package != 'openarm'}" column_inertial="${lift_inertial}"/>
+                               emit_arm_mounts="${arm_package != 'openarm'}" column_inertial="${lift_inertial}"
+                               column_geometry="${dict(section_x=lift_section[0], section_y=lift_section[1])}"/>
   <!-- so101: stub only. A9 (Jonathan) owns everything below so101_mount_link; nothing else is emitted for it here.
        none: the upper body only. -->

File: ros2/src/openamrobot_upperbody_description/urdf/openamrobot_upperbody.xacro (robot description, xacro)
@@ -19,8 +19,14 @@
                      {mass, com_z, ixx, iyy, izz}: it carries that inertial (the
                      combined robot supplies the sourced catalogue mass).
+    column_geometry  '' (none): the column has no visual and no collision. A dict
+                     {section_x, section_y}: both stages get a box of that section,
+                     visual and collision, named placeholder_*: the fixed stage on
+                     lift_column_base_link (retracted length), the moving stage on
+                     lift_carriage_link (stroke, below the carriage). Placeholder
+                     until the supplier drawing (datum lift_column_section).
 -->
 <robot xmlns:xacro="http://www.ros.org/wiki/xacro">
   <xacro:macro name="openamrobot_upperbody"
-      params="parent column base_plate head_pitch base_tilt column_axis_x_bp000 emit_arm_mounts:=true column_inertial:=''">
+      params="parent column base_plate head_pitch base_tilt column_axis_x_bp000 emit_arm_mounts:=true column_inertial:='' column_geometry:=''">
     <xacro:property name="cfg" lazy_eval="false"
         value="${xacro.load_yaml('$(find openamrobot_upperbody_description)/config/upperbody_configuration.yaml')}"/>
@@ -59,4 +65,14 @@
         </inertial>
       </xacro:unless>
+      <xacro:unless value="${column_geometry == ''}">
+        <visual name="placeholder_lift_column_fixed_stage">
+          <origin xyz="0 0 ${col['retracted_length'] / 2}" rpy="0 0 0"/>
+          <geometry><box size="${column_geometry['section_x']} ${column_geometry['section_y']} ${col['retracted_length']}"/></geometry>
+        </visual>
+        <collision name="placeholder_lift_column_fixed_stage">
+          <origin xyz="0 0 ${col['retracted_length'] / 2}" rpy="0 0 0"/>
+          <geometry><box size="${column_geometry['section_x']} ${column_geometry['section_y']} ${col['retracted_length']}"/></geometry>
+        </collision>
+      </xacro:unless>
     </link>
     <joint name="lift_column_base_joint" type="fixed">
@@ -68,5 +84,19 @@
          height is joint state. Effort and velocity limits are pending: they are
          set to 0 so the model cannot be used to command the lift. -->
-    <link name="lift_carriage_link"/>
+    <xacro:if value="${column_geometry == ''}">
+      <link name="lift_carriage_link"/>
+    </xacro:if>
+    <xacro:unless value="${column_geometry == ''}">
+      <link name="lift_carriage_link">
+        <visual name="placeholder_lift_column_moving_stage">
+          <origin xyz="0 0 ${-col['stroke'] / 2}" rpy="0 0 0"/>
+          <geometry><box size="${column_geometry['section_x']} ${column_geometry['section_y']} ${col['stroke']}"/></geometry>
+        </visual>
+        <collision name="placeholder_lift_column_moving_stage">
+          <origin xyz="0 0 ${-col['stroke'] / 2}" rpy="0 0 0"/>
+          <geometry><box size="${column_geometry['section_x']} ${column_geometry['section_y']} ${col['stroke']}"/></geometry>
+        </collision>
+      </link>
+    </xacro:unless>
     <joint name="lift_joint" type="prismatic">
       <parent link="lift_column_base_link"/>
