Commit message: feat(description): upper-body sensor frames, planar base joint and enforced frame contract
Add the S4 content of openamrobot_upperbody_description (part of #7):

- urdf/upper_sensors.xacro, emitted for arm_package == openarm: head camera
  on mast_mount_link and a wrist camera on each openarm_*_ee_base_link, each
  with a REP-103 optical frame, poses from the head/wrist camera datums.
  Marker-box visual only: no collision, no inertial (collision_free: true in
  the frame contract, with the reason). Plain frames; the ZED wrapper stays
  deferred.
- SO-101 stub: so101_mount_joint/link at identity on mast_mount_link; A9 owns
  everything below it.
- Planar base joint, emitted only with enable_planar_base:=true, under the
  A6 comment (disabled by default, AD-30): world link + base_planar_joint
  (planar, world -> base_link, axis z). The arg quoting in
  combined_robot.xacro is unchanged and now guarded by a test.
- frame_contract.yaml: base_link gets `variants` (root by default, planar
  child of world with enable_planar_base == true) so the contract is right
  in every expansion; collision_free fields on the three camera links.
- datums.yaml: the three pending_reference entries are deleted in this
  commit, which references those datums; revision 2026-10-08.c.
- T04: every expansion of the T01 matrix plus the planar flag honours the
  contract (R/C/W, parent and type, unlisted frames in our namespaces fail),
  missing W frames go to a JSON sidecar as a WARN. The checker is tested on
  synthetic URDFs.
- T11: no world/planar joint by default; correct when enabled; comment block
  present in the source. Sensor and so101 stub tests.
- view.launch.py gains enable_planar_base.

ros2_control is not emitted yet.

Assisted-by: Claude Code
Signed-off-by: Tushar Goel <Slash8860300674@gmail.com>

File: ros2/src/openamrobot_upperbody_description/urdf/combined_robot.xacro (robot description, xacro)
@@ -6,6 +6,9 @@
            -> mast_{left,right}_arm_mount_link                  (declared by the upstream macro, see below)
                 -> openarm_{left,right}_* arms + grippers        (upstream openarm_v20_robot, one call per arm)
-  Not here yet: ros2_control, sensors, the planar base joint. hardware_profile and enable_planar_base are
-  validated but have no effect until those land.
+                     -> {left,right}_wrist_camera_*              (upper_sensors.xacro)
+           -> head_camera_link / head_camera_optical_frame       (upper_sensors.xacro, on mast_mount_link)
+           -> so101_mount_link                                   (arm_package == so101: stub, A9 owns the rest)
+    world -> base_planar_joint -> base_link                      (only with enable_planar_base:=true)
+  Not here yet: ros2_control. hardware_profile is validated but has no effect until it lands.
   Args: an unknown value for any arg fails expansion with the list of accepted values.
 -->
@@ -41,14 +44,30 @@
                     value="${xacro.warning('hardware_profile:=' + hardware_profile + ' is accepted but has no effect yet: no ros2_control is emitted')}"/>
   </xacro:unless>
-  <xacro:if value="${enable_planar_base == 'true'}">
-    <xacro:property name="openamr_planar_base_inert" lazy_eval="false"
-                    value="${xacro.warning('enable_planar_base:=true is accepted but has no effect yet: no planar joint is emitted')}"/>
-  </xacro:if>
   <!-- Base: a full <robot> file from platform-sw, included unchanged; xacro merges its content. -->
   <xacro:include filename="$(find openamrobot_description)/urdf/robo_urdf.urdf.xacro"/>
+  <!-- A6: planar base joint — present, DISABLED by default (AD-30: base and arm never move together in OpenAMRobot 2.0). Enable only for future whole-body planning experiments. -->
+  <xacro:if value="${enable_planar_base == 'true'}">
+    <link name="world"/>
+    <!-- A planar joint moves in the plane normal to its axis; the URDF default axis is x, so z is set explicitly. -->
+    <joint name="base_planar_joint" type="planar">
+      <parent link="world"/>
+      <child link="base_link"/>
+      <origin xyz="0 0 0" rpy="0 0 0"/>
+      <axis xyz="0 0 1"/>
+    </joint>
+  </xacro:if>
   <xacro:include filename="$(find openamrobot_upperbody_description)/urdf/mast.xacro"/>
   <xacro:openamr_mast mast_id="${mast_id}" datums="${datums}" mast_ids="${mast_ids}"
                       arm_mounts="${arm_package == 'openarm'}"/>
-  <!-- so101: A9 owns it and nothing is emitted here. none: mast only. -->
+  <!-- so101: stub only. A9 (Jonathan) owns everything below so101_mount_link; nothing else is emitted for it here.
+       none: mast only. -->
+  <xacro:if value="${arm_package == 'so101'}">
+    <link name="so101_mount_link"/>
+    <joint name="so101_mount_joint" type="fixed">
+      <parent link="mast_mount_link"/>
+      <child link="so101_mount_link"/>
+      <origin xyz="0 0 0" rpy="0 0 0"/>
+    </joint>
+  </xacro:if>
   <xacro:if value="${arm_package == 'openarm'}">
     <xacro:include filename="$(find openarm_description)/assets/robot/openarm_v2.0/urdf/utils/openarm_v20_robot.xacro"/>
@@ -62,4 +81,7 @@
     <xacro:openarm_v20_robot config_root="${openarm_config_root}" robot_preset="${xacro.load_yaml(right_preset_file)}"
                              collapse_internal_empty_links="true" emit_grasp_frame="true"/>
+    <!-- Needs the openarm_*_ee_base_link links the two calls above emit. -->
+    <xacro:include filename="$(find openamrobot_upperbody_description)/urdf/upper_sensors.xacro"/>
+    <xacro:openamr_upper_sensors datums="${datums}"/>
   </xacro:if>
 </robot>

Commit message: feat(description): arm ros2_control profiles for mock, gazebo and real
urdf/ros2_control.xacro defines openamr_arm_ros2_control(hardware_profile),
called from combined_robot.xacro for arm_package:=openarm only. The base never
gets a <ros2_control> block (ADR-003).

- mock and real call upstream openarm_bimanual_ros2_control as upstream's own
  top-level v2.0 file does (same gains file, same finger-mimic file, same
  prefixes); use_fake_hardware follows the profile. The two blocks are equal,
  whitespace aside, to that file's expansion, and T14 and T16 assert it.
- gazebo emits our own system block, gz_ros2_control/GazeboSimSystem, for the
  same joints and the same command and state interfaces the upstream macro
  declares. finger_joint2 is left out as upstream leaves it out; whether
  gz_ros2_control needs a mimic parameter there is a TODO.

hardware_profile no longer prints "no effect yet" for a non-mock value.

T14 (mock: GenericSystem, no OpenArmHW, no base ros2_control, JTC interfaces
exported), T15 (gazebo) and T16 (real: OpenArmHW and CAN parameters, gains from
the upstream file) are expansion checks.

Assisted-by: Claude Code
Signed-off-by: Tushar Goel <Slash8860300674@gmail.com>

File: ros2/src/openamrobot_upperbody_description/urdf/combined_robot.xacro (robot description, xacro)
@@ -10,5 +10,6 @@
            -> so101_mount_link                                   (arm_package == so101: stub, A9 owns the rest)
     world -> base_planar_joint -> base_link                      (only with enable_planar_base:=true)
-  Not here yet: ros2_control. hardware_profile is validated but has no effect until it lands.
+  ros2_control (ros2_control.xacro): arms only, none for the base. hardware_profile picks the arm plugin: mock =
+  mock_components/GenericSystem, gazebo = gz_ros2_control/GazeboSimSystem, real = openarm_hardware/OpenArmHW (ADR-003).
   Args: an unknown value for any arg fails expansion with the list of accepted values.
 -->
@@ -40,8 +41,4 @@
   <xacro:openamr_require_one_of arg="hardware_profile" value="'${hardware_profile}'" accepted="${['mock', 'gazebo', 'real']}"/>
   <xacro:openamr_require_one_of arg="enable_planar_base" value="'${enable_planar_base}'" accepted="${['true', 'false']}"/>
-  <xacro:unless value="${hardware_profile == 'mock'}">
-    <xacro:property name="openamr_hardware_profile_inert" lazy_eval="false"
-                    value="${xacro.warning('hardware_profile:=' + hardware_profile + ' is accepted but has no effect yet: no ros2_control is emitted')}"/>
-  </xacro:unless>
   <!-- Base: a full <robot> file from platform-sw, included unchanged; xacro merges its content. -->
   <xacro:include filename="$(find openamrobot_description)/urdf/robo_urdf.urdf.xacro"/>
@@ -84,4 +81,7 @@
     <xacro:include filename="$(find openamrobot_upperbody_description)/urdf/upper_sensors.xacro"/>
     <xacro:openamr_upper_sensors datums="${datums}"/>
+    <!-- Arms only, and only here: so101 and none get no ros2_control. Needs the arm joints emitted above. -->
+    <xacro:include filename="$(find openamrobot_upperbody_description)/urdf/ros2_control.xacro"/>
+    <xacro:openamr_arm_ros2_control hardware_profile="${hardware_profile}"/>
   </xacro:if>
 </robot>

Commit message: refactor(description): the gazebo plugin's controller file is a xacro arg, not a $(find) of the control package
The description declares the hardware contract and knows nothing about where a controller
config lives (ADR-003). controllers_file defaults to empty, and the gazebo branch emits no
<parameters> when it is empty; sim.launch.py, which legitimately depends on both packages,
supplies the absolute path. That removes the colcon cycle instead of declaring it. T15
asserts the element appears when the arg is given, that the expansion is valid URDF when it
is not, that mock and real ignore the arg, and that no file here resolves the control package.

13 of the 14 expansions of the matrix are byte-identical before and after; the gazebo one
differs by the removed <parameters> line only.

Assisted-by: Claude Code
Signed-off-by: Tushar Goel <Slash8860300674@gmail.com>

File: ros2/src/openamrobot_upperbody_description/urdf/combined_robot.xacro (robot description, xacro)
@@ -20,4 +20,8 @@
   <xacro:arg name="enable_planar_base" default="false"/>
   <xacro:arg name="datums_file" default="$(find openamrobot_upperbody_description)/config/datums.yaml"/>
+  <!-- Absolute path of the controller parameter file the gazebo profile hands to gz_ros2_control. Empty by default: the
+       description declares the hardware contract and knows nothing about where a controller config lives (ADR-003); the launch
+       that starts the simulation supplies it. Only the gazebo profile reads it. -->
+  <xacro:arg name="controllers_file" default=""/>
   <!-- Args are read as raw strings: xacro would otherwise turn "false"/"true" (any case) and numerals into
        bool/number, and the accepted-value check below compares strings. The quotes + lazy_eval="false" keep them str. -->
@@ -27,4 +31,5 @@
   <xacro:property name="enable_planar_base" lazy_eval="false" value="'$(arg enable_planar_base)'"/>
   <xacro:property name="datums_file" lazy_eval="false" value="'$(arg datums_file)'"/>
+  <xacro:property name="controllers_file" lazy_eval="false" value="'$(arg controllers_file)'"/>
   <xacro:property name="mast_ids_file" value="$(find openamrobot_upperbody_description)/config/mast_ids.yaml"/>
   <xacro:property name="datums" value="${xacro.load_yaml(datums_file)}"/>
@@ -83,5 +88,5 @@
     <!-- Arms only, and only here: so101 and none get no ros2_control. Needs the arm joints emitted above. -->
     <xacro:include filename="$(find openamrobot_upperbody_description)/urdf/ros2_control.xacro"/>
-    <xacro:openamr_arm_ros2_control hardware_profile="${hardware_profile}"/>
+    <xacro:openamr_arm_ros2_control hardware_profile="${hardware_profile}" controllers_file="${controllers_file}"/>
   </xacro:if>
 </robot>

File: ros2/src/openamrobot_upperbody_description/urdf/ros2_control.xacro (robot description, xacro)
@@ -43,5 +43,5 @@
     </joint>
   </xacro:macro>
-  <xacro:macro name="openamr_arm_ros2_control" params="hardware_profile">
+  <xacro:macro name="openamr_arm_ros2_control" params="hardware_profile controllers_file:=''">
     <xacro:if value="${hardware_profile in ['mock', 'real']}">
       <!-- What upstream's openarm_v20.urdf.xacro does before it calls the macro. -->
@@ -66,9 +66,14 @@
            read from the installed Jazzy gz_ros2_control 1.2.20, not from documentation: libgz_ros2_control-system.so
            registers gz_ros2_control::GazeboSimROS2ControlPlugin (libgz_hardware_plugins.so registers GazeboSimSystem).
-           The controllers are the same file every profile uses (ADR-003). The world, physics, sensors and the launch that
-           spawns this model are simulation bringup and live in openamrobot_upperbody_gazebo. -->
+           The controllers are the same file every profile uses (ADR-003), but this description does not know where it lives:
+           the path comes in as the controllers_file arg, and with the arg empty (the default) there is no <parameters> at all.
+           The launch that starts the simulation supplies it, so this package does not resolve the control package's path
+           (it would be an undeclared dependency, or a cycle: control test-depends on this package). The world, physics,
+           sensors and the launch that spawns this model are simulation bringup and live in openamrobot_upperbody_gazebo. -->
       <gazebo>
         <plugin filename="gz_ros2_control-system" name="gz_ros2_control::GazeboSimROS2ControlPlugin">
-          <parameters>$(find openamrobot_upperbody_control)/config/arm_controllers.yaml</parameters>
+          <xacro:if value="${controllers_file != ''}">
+            <parameters>${controllers_file}</parameters>
+          </xacro:if>
         </plugin>
       </gazebo>
