Commit message: feat(description)!: adopt option B in the combined robot, delete the mast, rev19.0 numbers
The combined robot is option B's upper body (lift column, prismatic lift_joint, carriage, arm
profile, head camera) on platform-sw's base_footprint, plus what composition adds. No mast:
urdf/mast.xacro, config/mast_ids.yaml and the datums mast_base_pose, left/right_arm_mount_pose,
mast_section, mast_mass and head_camera_pose are deleted, and mast_id is not an argument.

* The arms are rooted on option B's mount frames: two calls of the macro that openarm_v20_robot
  itself calls (it declares its root_frame as a link, which would duplicate lift_carriage_link),
  with the mount pose read from upperbody_configuration.yaml. ADR-008 is otherwise unchanged:
  two calls, derived single-arm presets, no OpenArm body.
* rev19.0 numbers: two base plates (bp000, bp050); the column axis at x +0.060 / +0.110 from
  base_link, not on the drive axle (datum column_axis_x_bp000); base_link_height_above_floor
  0.098 (was a placeholder since S3), asserted equal to platform-sw's base_footprint_joint;
  the lift 11.7 kg catalogue (DOLD Hexalift V4 350) on lift_column_base_link.
* Three option-B adoptions: effort 0 / velocity 0 on the lift joint, kept; a null datum is a
  hard-fail naming itself (lift_mass_tl3_400, as option B's tl3_400 lengths); calibration IDs
  (the lift stops L1000/L1175/L1350, joint positions) are not configuration IDs.
* config_id inputs: column, base_plate, head_pitch, base_tilt, arm_package, hardware_profile,
  datums revision, every upstream pin, and the canonical URDF. mast_id leaves. The format is
  unchanged and valid against C9; the meaning is not, and nothing will say so.
* Frame contract: the base is base_footprint -> base_link; the six near-field frames
  (tof_front_left_link ... ultrasonic_rear_link, declared and absent: T04's WARN) are REMOVED,
  not renamed: platform-sw declares us_* and tof_* (935efc7) and the contract says they are
  consumed from there. T04 PASS, W01 PASS (the root carries no inertial).
* Datum rules from V01: a dimension list declares axis_convention and T12 asserts the
  assignment; a mass of ours declares a density_band and T10 reports the implied density.
* T05 is shoulder height per lift stop; E01 is per lift stop; T10 drops the mast group and
  gains the lift; the expansion matrix is one factor at a time around the baseline (14).

Assisted-by: Claude Code
Signed-off-by: Tushar Goel <Slash8860300674@gmail.com>

File: ros2/src/openamrobot_upperbody_description/urdf/combined_robot.xacro (robot description, xacro)
@@ -1,19 +1,31 @@
 <?xml version="1.0"?>
 <!--
-  OpenAMRobot 2.0 combined robot description (ARCHITECTURE.md s3-5, ADR-001/004/005/006/008).
-    base_link (platform-sw, included unchanged)
-      -> mast_base_link -> mast_mount_link                      (mast.xacro, datums + mast_ids)
-           -> mast_{left,right}_arm_mount_link                  (declared by the upstream macro, see below)
-                -> openarm_{left,right}_* arms + grippers        (upstream openarm_v20_robot, one call per arm)
-                     -> {left,right}_wrist_camera_*              (upper_sensors.xacro)
-           -> head_camera_link / head_camera_optical_frame       (upper_sensors.xacro, on mast_mount_link)
-           -> so101_mount_link                                   (arm_package == so101: stub, A9 owns the rest)
-    world -> base_planar_joint -> base_link                      (only with enable_planar_base:=true)
-  ros2_control (ros2_control.xacro): arms only, none for the base. hardware_profile picks the arm plugin: mock =
-  mock_components/GenericSystem, gazebo = gz_ros2_control/GazeboSimSystem, real = openarm_hardware/OpenArmHW (ADR-003).
-  Args: an unknown value for any arg fails expansion with the list of accepted values.
+  OpenAMRobot 2.0 combined robot description (ARCHITECTURE.md s3-5, ADR-001/004/005/008/010, P-03 rev19.0).
+    base_footprint (platform-sw: the root, on the floor under the drive-axle midpoint, REP 105)
+      -> base_link (platform-sw, 0.098 m above it) and everything platform-sw declares on it, near-field frames included
+      -> lift_column_base_link                                  (option B, openamrobot_upperbody.xacro; datum column_axis_x_bp000)
+           -> lift_joint (prismatic, 0..0.350 m, effort 0 velocity 0: no authority to command it) -> lift_carriage_link
+                -> arm_profile_link
+                -> head_camera_mount_link -> head_camera_link -> head_camera_optical_frame     (option B)
+                -> openarm_{left,right}_base_link                (declared by the upstream arm macro, at option B's mount pose)
+                     -> openarm_{left,right}_* arms + grippers   (upstream, one call per arm; ADR-008)
+                          -> {left,right}_wrist_camera_*         (upper_sensors.xacro)
+                -> so101_mount_link                              (arm_package == so101: stub, A9 owns the rest)
+    world -> base_planar_joint -> base_footprint                 (only with enable_planar_base:=true)
+  The upper-body geometry is Alex's (option B, merged on main) and is consumed, not rewritten. Everything this file adds is the
+  composition: the arms, the lift column's inertial (datums), the sensors on the wrists, ros2_control. No mast: the shoulder
+  height is the joint position of lift_joint (calibration IDs L1000 / L1175 / L1350 are joint positions, not arguments).
+  ros2_control (ros2_control.xacro): arms only, none for the base and none for the lift. hardware_profile picks the arm plugin:
+  mock = mock_components/GenericSystem, gazebo = gz_ros2_control/GazeboSimSystem, real = openarm_hardware/OpenArmHW (ADR-003).
+  Args: an unknown value for any arg fails expansion with the list of accepted values. column, base_plate, head_pitch and
+  base_tilt are option B's configuration IDs; their accepted values and baseline are read from upperbody_configuration.yaml.
+  A configuration whose supplier data is null (column tl3_400) does not expand; neither does a null datum that is read.
 -->
 <robot xmlns:xacro="http://www.ros.org/wiki/xacro" name="openamrobot">
-  <xacro:arg name="mast_id" default="mast_1350"/>
+  <!-- The defaults are option B's baseline; T01 asserts they equal upperbody_configuration.yaml's `baseline:`. -->
+  <xacro:arg name="column" default="dold_v4_350"/>
+  <xacro:arg name="base_plate" default="bp000"/>
+  <xacro:arg name="head_pitch" default="hp25"/>
+  <xacro:arg name="base_tilt" default="bt10"/>
   <xacro:arg name="arm_package" default="openarm"/>
   <xacro:arg name="hardware_profile" default="mock"/>
@@ -26,5 +38,8 @@
   <!-- Args are read as raw strings: xacro would otherwise turn "false"/"true" (any case) and numerals into
        bool/number, and the accepted-value check below compares strings. The quotes + lazy_eval="false" keep them str. -->
-  <xacro:property name="mast_id" lazy_eval="false" value="'$(arg mast_id)'"/>
+  <xacro:property name="column" lazy_eval="false" value="'$(arg column)'"/>
+  <xacro:property name="base_plate" lazy_eval="false" value="'$(arg base_plate)'"/>
+  <xacro:property name="head_pitch" lazy_eval="false" value="'$(arg head_pitch)'"/>
+  <xacro:property name="base_tilt" lazy_eval="false" value="'$(arg base_tilt)'"/>
   <xacro:property name="arm_package" lazy_eval="false" value="'$(arg arm_package)'"/>
   <xacro:property name="hardware_profile" lazy_eval="false" value="'$(arg hardware_profile)'"/>
@@ -32,7 +47,7 @@
   <xacro:property name="datums_file" lazy_eval="false" value="'$(arg datums_file)'"/>
   <xacro:property name="controllers_file" lazy_eval="false" value="'$(arg controllers_file)'"/>
-  <xacro:property name="mast_ids_file" value="$(find openamrobot_upperbody_description)/config/mast_ids.yaml"/>
   <xacro:property name="datums" value="${xacro.load_yaml(datums_file)}"/>
-  <xacro:property name="mast_ids" value="${xacro.load_yaml(mast_ids_file)}"/>
+  <xacro:property name="upperbody" lazy_eval="false"
+                  value="${xacro.load_yaml('$(find openamrobot_upperbody_description)/config/upperbody_configuration.yaml')}"/>
   <!-- Arg validation: xacro.fatal() raises XacroException carrying this message (no Python traceback to read). -->
   <xacro:macro name="openamr_require_one_of" params="arg value accepted">
@@ -42,9 +57,14 @@
     </xacro:unless>
   </xacro:macro>
-  <xacro:openamr_require_one_of arg="mast_id" value="'${mast_id}'" accepted="${list(mast_ids['mast_ids'].keys())}"/>
+  <xacro:openamr_require_one_of arg="column" value="'${column}'" accepted="${upperbody['configuration_axes']['column']}"/>
+  <xacro:openamr_require_one_of arg="base_plate" value="'${base_plate}'" accepted="${upperbody['configuration_axes']['base_plate']}"/>
+  <xacro:openamr_require_one_of arg="head_pitch" value="'${head_pitch}'" accepted="${upperbody['configuration_axes']['head_pitch']}"/>
+  <xacro:openamr_require_one_of arg="base_tilt" value="'${base_tilt}'" accepted="${upperbody['configuration_axes']['base_tilt']}"/>
   <xacro:openamr_require_one_of arg="arm_package" value="'${arm_package}'" accepted="${['openarm', 'so101', 'none']}"/>
   <xacro:openamr_require_one_of arg="hardware_profile" value="'${hardware_profile}'" accepted="${['mock', 'gazebo', 'real']}"/>
   <xacro:openamr_require_one_of arg="enable_planar_base" value="'${enable_planar_base}'" accepted="${['true', 'false']}"/>
-  <!-- Base: a full <robot> file from platform-sw, included unchanged; xacro merges its content. -->
+  <!-- Base: a full <robot> file from platform-sw, included unchanged; xacro merges its content. Since platform-sw 935efc7 its
+       root is base_footprint (REP 105) and it declares the near-field frames, the base camera and the IMU: none of those is
+       declared here (ADR-010 s4/s5 and the frame contract). It also declares the base_tilt arg, which is the same arg as above. -->
   <xacro:include filename="$(find openamrobot_description)/urdf/robo_urdf.urdf.xacro"/>
   <!-- A6: planar base joint — present, DISABLED by default (AD-30: base and arm never move together in OpenAMRobot 2.0). Enable only for future whole-body planning experiments. -->
@@ -54,18 +74,49 @@
     <joint name="base_planar_joint" type="planar">
       <parent link="world"/>
-      <child link="base_link"/>
+      <child link="base_footprint"/>
       <origin xyz="0 0 0" rpy="0 0 0"/>
       <axis xyz="0 0 1"/>
     </joint>
   </xacro:if>
-  <xacro:include filename="$(find openamrobot_upperbody_description)/urdf/mast.xacro"/>
-  <xacro:openamr_mast mast_id="${mast_id}" datums="${datums}" mast_ids="${mast_ids}"
-                      arm_mounts="${arm_package == 'openarm'}"/>
+  <!-- Datums are read through these properties. A null datum stops the expansion and names itself. -->
+  <xacro:property name="dt" value="${datums['datums']}"/>
+  <xacro:macro name="openamr_require_datum" params="name value owner">
+    <xacro:if value="${value is None}">
+      <xacro:property name="openamr_datum_null_${name}" lazy_eval="false"
+                      value="${xacro.fatal('datum ' + name + ' is null (supplier data that does not exist yet; owner: ' + owner + '): this configuration cannot be built, and nothing is guessed in its place')}"/>
+    </xacro:if>
+  </xacro:macro>
+  <!-- The lift column's inertial. Mass: the catalogue figure of the selected column, a datum per column (hard-fail when null).
+       Shape: a uniform box of the column's section (datum, axis convention x fore-aft, y lateral) and its retracted length (option B's
+       config), centred at half of that length above lift_column_base_link. All of the mass is on the fixed side (the catalogue
+       does not split it). No collision and no visual: the column body's lateral extent is not sourced. -->
+  <xacro:property name="lift_mass_by_column" lazy_eval="false"
+                  value="${dict(dold_v4_350=dt['lift_mass_dold_v4_350']['value'], tl3_400=dt['lift_mass_tl3_400']['value'])}"/>
+  <xacro:property name="lift_mass" lazy_eval="false" value="${lift_mass_by_column[column]}"/>
+  <xacro:openamr_require_datum name="lift_mass_${column}" value="${lift_mass}" owner="Alex (F2S)"/>
+  <xacro:property name="column_cfg" lazy_eval="false" value="${upperbody['column'][column]}"/>
+  <xacro:if value="${column_cfg['retracted_length'] is None}">
+    ${xacro.fatal("column '" + column + "': retracted length is pending supplier data; this configuration cannot be built yet")}
+  </xacro:if>
+  <xacro:property name="lift_section" lazy_eval="false" value="${dt['lift_column_section']['value']}"/>
+  <xacro:property name="lift_h" lazy_eval="false" value="${column_cfg['retracted_length']}"/>
+  <xacro:property name="lift_inertial" lazy_eval="false"
+                  value="${dict(mass=lift_mass, com_z=lift_h / 2,
+                                ixx=lift_mass * (lift_section[1] * lift_section[1] + lift_h * lift_h) / 12,
+                                iyy=lift_mass * (lift_section[0] * lift_section[0] + lift_h * lift_h) / 12,
+                                izz=lift_mass * (lift_section[0] * lift_section[0] + lift_section[1] * lift_section[1]) / 12)}"/>
+  <!-- Option B's upper body, on base_footprint: its heights are from the floor. With arm_package == openarm the upstream macro below
+       declares openarm_{left,right}_base_link and their mount joints at the same pose (emit_arm_mounts false); with none or so101
+       the mount frames are option B's own, so every expansion has them. -->
+  <xacro:include filename="$(find openamrobot_upperbody_description)/urdf/openamrobot_upperbody.xacro"/>
+  <xacro:openamrobot_upperbody parent="base_footprint" column="${column}" base_plate="${base_plate}" head_pitch="${head_pitch}"
+                               base_tilt="${base_tilt}" column_axis_x_bp000="${dt['column_axis_x_bp000']['value']}"
+                               emit_arm_mounts="${arm_package != 'openarm'}" column_inertial="${lift_inertial}"/>
   <!-- so101: stub only. A9 (Jonathan) owns everything below so101_mount_link; nothing else is emitted for it here.
-       none: mast only. -->
+       none: the upper body only. -->
   <xacro:if value="${arm_package == 'so101'}">
     <link name="so101_mount_link"/>
     <joint name="so101_mount_joint" type="fixed">
-      <parent link="mast_mount_link"/>
+      <parent link="lift_carriage_link"/>
       <child link="so101_mount_link"/>
       <origin xyz="0 0 0" rpy="0 0 0"/>
@@ -77,10 +128,28 @@
     <xacro:property name="left_preset_file" value="$(find openamrobot_upperbody_description)/config/openarm_preset_left.yaml"/>
     <xacro:property name="right_preset_file" value="$(find openamrobot_upperbody_description)/config/openarm_preset_right.yaml"/>
-    <!-- ADR-008: no OpenArm body. One macro call per arm, each rooted on its mast plate link.
-         Upstream rejects two enabled root components, so the bimanual preset cannot be reparented. -->
-    <xacro:openarm_v20_robot config_root="${openarm_config_root}" robot_preset="${xacro.load_yaml(left_preset_file)}"
-                             collapse_internal_empty_links="true" emit_grasp_frame="true"/>
-    <xacro:openarm_v20_robot config_root="${openarm_config_root}" robot_preset="${xacro.load_yaml(right_preset_file)}"
-                             collapse_internal_empty_links="true" emit_grasp_frame="true"/>
+    <!-- ADR-008 (unchanged in kind): no OpenArm body, one call per arm, each on a derived single-arm preset (upstream rejects two
+         enabled root components, so the bimanual preset cannot be reparented). Two things differ from the mast version:
+           1. The arm's parent is option B's lift_carriage_link and its mount pose is option B's own: x from the column axis,
+              y +-, z above the column top, from upperbody_configuration.yaml geometry.arm_mount. The preset files keep upstream's
+              zero origin; the pose is set here so that there is one source for it.
+           2. openarm_v20_robot is not called: it declares the root_frame as a link, and option B already declares
+              lift_carriage_link (a second declaration is an invalid URDF). Its body is validate + that link + the macro below,
+              which is called as it calls it. Pinned to the upstream commit of config/upstream_pins.yaml (C02). -->
+    <xacro:property name="arm_mount" lazy_eval="false" value="${upperbody['geometry']['arm_mount']}"/>
+    <xacro:macro name="openamr_arm_preset" params="file sign">
+      <xacro:property name="preset" lazy_eval="false" value="${xacro.load_yaml(file)}"/>
+      <!-- A new dict, not an update(): xacro.load_yaml wraps every nested dict in a copy on access, so mutating one changes nothing. -->
+      <xacro:property name="preset_with_mount" lazy_eval="false"
+                      value="${dict(preset, primary_arm=dict(preset['primary_arm'], connection=dict(preset['primary_arm']['connection'],
+                                    origin=dict(x=arm_mount['x_from_column_axis'], y=sign * arm_mount['y'], z=arm_mount['z_above_column_top'],
+                                                roll=0.0, pitch=0.0, yaw=0.0))))}"/>
+      <xacro:openarm_v20_validate_robot_preset components="${preset_with_mount['robot']['components']}" robot_preset="${preset_with_mount}"/>
+      <xacro:openarm_v20_emit_attached_components index="0" components="${preset_with_mount['robot']['components']}"
+                                                  parent_component_name="__root__" robot_preset="${preset_with_mount}"
+                                                  config_root="${openarm_config_root}" root_frame="${preset_with_mount['robot']['root_frame']}"
+                                                  collapse_internal_empty_links="true" emit_grasp_frame="true"/>
+    </xacro:macro>
+    <xacro:openamr_arm_preset file="${left_preset_file}" sign="1"/>
+    <xacro:openamr_arm_preset file="${right_preset_file}" sign="-1"/>
     <!-- Needs the openarm_*_ee_base_link links the two calls above emit. -->
     <xacro:include filename="$(find openamrobot_upperbody_description)/urdf/upper_sensors.xacro"/>

File: ros2/src/openamrobot_upperbody_description/urdf/upper_sensors.xacro (robot description, xacro)
@@ -1,16 +1,22 @@
 <?xml version="1.0"?>
 <!--
-  Upper-body sensor frames (FRAMES.md, DESIGN_LOG 2026-09-21: plain frames, the ZED wrapper is deferred).
+  Upper-body sensor frames (FRAMES.md, DESIGN_LOG 2026-09-21: plain frames).
   Emitted by combined_robot.xacro when arm_package == 'openarm'.
-    head_camera_link           on mast_mount_link             pose = datum head_camera_pose
     left_wrist_camera_link     on openarm_left_ee_base_link   pose = datum left_wrist_camera_pose
     right_wrist_camera_link    on openarm_right_ee_base_link  pose = datum right_wrist_camera_pose
     each with a <name>_optical_frame child (REP-103: z forward, x right, y down)
+  The head camera is not here: option B declares head_camera_mount_link, head_camera_link and head_camera_optical_frame with
+  sourced numbers (ZED Mini lens offset, head_pitch), and this file's former head_camera_pose placeholder is deleted.
   Each camera link carries a small box VISUAL and no <collision> and no <inertial>: the box is a marker for where the
   frame is, not a model of the sensor. Frame contract entries say collision_free: true with the reason.
-  Needs mast.xacro included first (openamr_origin_from_pose). The parents of the wrist cameras are links of the
-  upstream openarm_v20_robot macro, so this file must be instantiated after both macro calls.
+  The parents of the wrist cameras are links of the upstream openarm_v20_robot macros, so this file must be instantiated
+  after both calls.
 -->
 <robot xmlns:xacro="http://www.ros.org/wiki/xacro">
+  <!-- <origin> from a datum pose {xyz: [x, y, z], rpy: [r, p, y]}. -->
+  <xacro:macro name="openamr_origin_from_pose" params="pose">
+    <origin xyz="${pose['xyz'][0]} ${pose['xyz'][1]} ${pose['xyz'][2]}"
+            rpy="${pose['rpy'][0]} ${pose['rpy'][1]} ${pose['rpy'][2]}"/>
+  </xacro:macro>
   <!-- Visualization constant (DATUMS.md): edge, in metres, of the marker box drawn for each camera frame. It describes
        how the model is drawn, not the robot, so it is not a datum. It may appear only inside a <visual>: no collision,
@@ -39,6 +45,4 @@
   <xacro:macro name="openamr_upper_sensors" params="datums">
     <xacro:property name="dt" value="${datums['datums']}"/>
-    <xacro:openamr_camera_frames name="head_camera" parent="mast_mount_link"
-                                 pose="${dt['head_camera_pose']['value']}"/>
     <xacro:openamr_camera_frames name="left_wrist_camera" parent="openarm_left_ee_base_link"
                                  pose="${dt['left_wrist_camera_pose']['value']}"/>
