Commit message: feat(description): lift column on the DOLD datasheet's sections, the carriage as the inner stage, the adapter plate as its own link (P28)
Alex, 22 Oct 2026 (P-03 rev19.6 item 18):
- lift_column_section is [0.240, 0.060], source supplier, status provisional, from the
  DOLD Hexalift datasheet page 4 ("Outer profile 240x60"); matches option B drawing
  sheet 2 rev A. The lateral side is no longer invented.
- the carriage is the Hexalift INNER stage: new datum lift_inner_section [0.2095, 0.051]
  (same drawing, "Inner profile 209.5x51"; supplier, provisional), strictly smaller than
  the outer on both axes. It was a second copy of the outer section. The stage length is
  still the stroke (the datasheet gives none); the outer collision is a solid box, so the
  volumes still overlap.
- the adapter plate, 360 x 100 x 10 mm (new datum adapter_plate_section, plan,
  provisional), is its own link on the carriage, rear edge flush with the column's rear
  face. arm_profile_link is its child (pose from the carriage unchanged): touching
  siblings were a permanent collision of the model in the derivation, a parent and child
  are a structural neighbour.

Consequences: the collision matrix is re-derived, 99 disabled pairs (20 upstream + 18
Adjacent + 61 ConstantTransform, was 95); the lift mass density band is re-fitted from
1200 to 1600 kg/m3 because the sourced section puts 11.7 kg at 1533 kg/m3 (judgement call,
reason in the datum); datums revision 2026-10-28.a. Tests: T10, T12, the P25 material
test and the ACM counts follow; test_p28_lift_geometry.py is new.

Assisted-by: Claude Code
Signed-off-by: Tushar Goel <Slash8860300674@gmail.com>

File: ros2/src/openamrobot_upperbody_description/urdf/combined_robot.xacro (robot description, xacro)
@@ -91,6 +91,7 @@
        Shape: a uniform box of the column's section (datum, axis convention x fore-aft, y lateral) and its retracted length (option B's
        config), centred at half of that length above lift_column_base_link. All of the mass is on the fixed side (the catalogue
-       does not split it). Visual and collision: placeholder boxes of the same section on both stages (column_geometry), until the
-       supplier drawing; the column body's lateral extent is not sourced. -->
+       does not split it). Visual and collision (column_geometry): the OUTER stage a box of lift_column_section on lift_column_base_link,
+       the INNER stage a box of lift_inner_section (strictly smaller, from the same DOLD datasheet page) on lift_carriage_link; the inner
+       stage's length is the stroke, which the datasheet does not give as a length. The adapter plate (adapter_plate_section) is its own link. -->
   <xacro:property name="lift_mass_by_column" lazy_eval="false"
                   value="${dict(dold_v4_350=dt['lift_mass_dold_v4_350']['value'], tl3_400=dt['lift_mass_tl3_400']['value'])}"/>
@@ -102,4 +103,6 @@
   </xacro:if>
   <xacro:property name="lift_section" lazy_eval="false" value="${dt['lift_column_section']['value']}"/>
+  <xacro:property name="lift_inner" lazy_eval="false" value="${dt['lift_inner_section']['value']}"/>
+  <xacro:property name="plate_section" lazy_eval="false" value="${dt['adapter_plate_section']['value']}"/>
   <xacro:property name="lift_h" lazy_eval="false" value="${column_cfg['retracted_length']}"/>
   <xacro:property name="lift_inertial" lazy_eval="false"
@@ -115,5 +118,6 @@
                                base_tilt="${base_tilt}" column_axis_x_bp000="${dt['column_axis_x_bp000']['value']}"
                                emit_arm_mounts="${arm_package != 'openarm'}" column_inertial="${lift_inertial}"
-                               column_geometry="${dict(section_x=lift_section[0], section_y=lift_section[1])}"/>
+                               column_geometry="${dict(section_x=lift_section[0], section_y=lift_section[1], inner_x=lift_inner[0], inner_y=lift_inner[1])}"
+                               adapter_plate="${dict(size_x=plate_section[0], size_y=plate_section[1], center_x=-lift_section[0] / 2 + plate_section[0] / 2)}"/>
   <!-- so101: stub only. A9 (Jonathan) owns everything below so101_mount_link; nothing else is emitted for it here.
        none: the upper body only. -->

File: ros2/src/openamrobot_upperbody_description/urdf/openamrobot_upperbody.xacro (robot description, xacro)
@@ -21,13 +21,21 @@
                      combined robot supplies the sourced catalogue mass).
     column_geometry  '' (none): the column has no visual and no collision. A dict
-                     {section_x, section_y}: both stages get a box of that section,
-                     visual and collision (the collisions named placeholder_*): the fixed stage on
-                     lift_column_base_link (retracted length), the moving stage on
-                     lift_carriage_link (stroke, below the carriage). Placeholder
-                     until the supplier drawing (datum lift_column_section).
+                     {section_x, section_y, inner_x, inner_y}: the two stages of the Hexalift,
+                     each a box, visual and collision (the collisions named placeholder_*): the
+                     OUTER (fixed) stage of section_x x section_y on lift_column_base_link
+                     (retracted length), the INNER (moving) stage of inner_x x inner_y on
+                     lift_carriage_link (stroke, below the carriage). The sections are the
+                     supplier's (datums lift_column_section and lift_inner_section); the
+                     inner stage's length is not, it is the stroke.
+    adapter_plate    '' (none): no adapter plate link. A dict {size_x, size_y, center_x}: the
+                     plate under the arm profile, its own link adapter_plate_link on
+                     lift_carriage_link, size_x fore-aft by size_y lateral by
+                     geometry.adapter_plate_thickness, resting on the carriage frame's
+                     horizontal plane (the column top at lift 0) and centred laterally;
+                     center_x is from the column axis (datum adapter_plate_section).
 -->
 <robot xmlns:xacro="http://www.ros.org/wiki/xacro">
   <xacro:macro name="openamrobot_upperbody"
-      params="parent column base_plate head_pitch base_tilt column_axis_x_bp000 emit_arm_mounts:=true column_inertial:='' column_geometry:=''">
+      params="parent column base_plate head_pitch base_tilt column_axis_x_bp000 emit_arm_mounts:=true column_inertial:='' column_geometry:='' adapter_plate:=''">
     <xacro:property name="cfg" lazy_eval="false"
         value="${xacro.load_yaml('$(find openamrobot_upperbody_description)/config/upperbody_configuration.yaml')}"/>
@@ -112,10 +120,10 @@
         <visual>
           <origin xyz="0 0 ${-col['stroke'] / 2}" rpy="0 0 0"/>
-          <geometry><box size="${column_geometry['section_x']} ${column_geometry['section_y']} ${col['stroke']}"/></geometry>
+          <geometry><box size="${column_geometry['inner_x']} ${column_geometry['inner_y']} ${col['stroke']}"/></geometry>
           <material name="placeholder_geometry"/>
         </visual>
         <collision name="placeholder_lift_column_moving_stage">
           <origin xyz="0 0 ${-col['stroke'] / 2}" rpy="0 0 0"/>
-          <geometry><box size="${column_geometry['section_x']} ${column_geometry['section_y']} ${col['stroke']}"/></geometry>
+          <geometry><box size="${column_geometry['inner_x']} ${column_geometry['inner_y']} ${col['stroke']}"/></geometry>
         </collision>
       </link>
@@ -129,4 +137,24 @@
       <limit lower="0.0" upper="${col['stroke']}" effort="0.0" velocity="0.0"/>
     </joint>
+    <!-- Adapter plate (P-03 rev19.6 item 18): its own link, carried by the carriage, under the arm profile. Its joint is at the box centre and
+         the link has no <origin>, the convention arm_profile_link uses. The plate rests on the carriage frame's horizontal plane (z 0 to the
+         thickness), so the profile's 10 mm offset below is its top face. -->
+    <xacro:unless value="${adapter_plate == ''}">
+      <link name="adapter_plate_link">
+        <visual>
+          <geometry><box size="${adapter_plate['size_x']} ${adapter_plate['size_y']} ${geo['adapter_plate_thickness']}"/></geometry>
+          <material name="placeholder_geometry"/>
+        </visual>
+        <collision name="adapter_plate">
+          <geometry><box size="${adapter_plate['size_x']} ${adapter_plate['size_y']} ${geo['adapter_plate_thickness']}"/></geometry>
+        </collision>
+      </link>
+      <xacro:openamrobot_placeholder_gazebo_material link="adapter_plate_link"/>
+      <joint name="adapter_plate_joint" type="fixed">
+        <parent link="lift_carriage_link"/>
+        <child link="adapter_plate_link"/>
+        <origin xyz="${adapter_plate['center_x']} 0 ${geo['adapter_plate_thickness'] / 2}" rpy="0 0 0"/>
+      </joint>
+    </xacro:unless>
     <!-- Arm profile (MISUMI HFS6-60120) on the adapter plate. -->
     <link name="arm_profile_link">
@@ -140,9 +168,21 @@
     </link>
     <xacro:openamrobot_placeholder_gazebo_material link="arm_profile_link"/>
-    <joint name="arm_profile_joint" type="fixed">
-      <parent link="lift_carriage_link"/>
-      <child link="arm_profile_link"/>
-      <origin xyz="${profile['center_x_from_column_axis']} 0 ${geo['adapter_plate_thickness'] + profile['length'] / 2}" rpy="0 0 0"/>
-    </joint>
+    <!-- With the adapter plate modelled the profile hangs off the plate it stands on (P28): the two faces touch by design (the profile's bottom
+         face is the plate's top face), and two siblings that touch would be a permanent collision of the model, where a parent and its child are
+         a structural neighbour. The profile's pose from the carriage is the same either way: x center_x_from_column_axis, z thickness + length / 2. -->
+    <xacro:if value="${adapter_plate == ''}">
+      <joint name="arm_profile_joint" type="fixed">
+        <parent link="lift_carriage_link"/>
+        <child link="arm_profile_link"/>
+        <origin xyz="${profile['center_x_from_column_axis']} 0 ${geo['adapter_plate_thickness'] + profile['length'] / 2}" rpy="0 0 0"/>
+      </joint>
+    </xacro:if>
+    <xacro:unless value="${adapter_plate == ''}">
+      <joint name="arm_profile_joint" type="fixed">
+        <parent link="adapter_plate_link"/>
+        <child link="arm_profile_link"/>
+        <origin xyz="${profile['center_x_from_column_axis'] - adapter_plate['center_x']} 0 ${geo['adapter_plate_thickness'] / 2 + profile['length'] / 2}" rpy="0 0 0"/>
+      </joint>
+    </xacro:unless>
     <!-- OpenArm J1_A arm mount points. -->
     <xacro:macro name="openamrobot_arm_mount" params="side sign">
