Commit message: feat(description): two opt-in parameters on option B's macro, so the combined robot can compose it
Option B declares openarm_{left,right}_base_link and a mount joint of the same name as
upstream's arm macro emits (openarm_left_base_link_mount_joint): the arm's base link IS its
mount frame, so declaring both is a duplicate link and an invalid URDF. The macro gains
emit_arm_mounts (default true) so that the combined robot can have the upstream arm macro
emit them at the same pose, and column_inertial (default none) so that the lift's catalogue
mass can sit on lift_column_base_link: option B models no masses.

Both default to its own behaviour. With neither given the macro expands exactly as on
upstream/main, and the standalone wrapper is untouched; test_t04_optb_composition.py asserts
both. Not re-authoring anything: this is a new commit on top of Alex's two, and it is a
change for him and Cuma to accept or to ask us to carry some other way.

Assisted-by: Claude Code
Signed-off-by: Tushar Goel <Slash8860300674@gmail.com>

File: ros2/src/openamrobot_upperbody_description/urdf/openamrobot_upperbody.xacro (robot description, xacro)
@@ -8,8 +8,19 @@
   All values come from config/upperbody_configuration.yaml. No masses, inertias
   or supplier outlines are modelled: they are pending supplier CAD.
+  Two opt-in parameters let the combined robot (combined_robot.xacro) compose this
+  model with the upstream OpenArm macro. Both default to this file's own behaviour:
+    emit_arm_mounts  true: declare openarm_{left,right}_base_link and their mount
+                     joints (frames only, as before). false: declare neither. The
+                     upstream arm macro emits a link and a joint of exactly those
+                     names, with the arm's own geometry, so declaring them here as
+                     well would duplicate them; the combined robot sets false and
+                     gives the upstream macro the same parent and origin.
+    column_inertial  '' (none): lift_column_base_link carries no inertial. A dict
+                     {mass, com_z, ixx, iyy, izz}: it carries that inertial (the
+                     combined robot supplies the sourced catalogue mass).
 -->
 <robot xmlns:xacro="http://www.ros.org/wiki/xacro">
   <xacro:macro name="openamrobot_upperbody"
-      params="parent column base_plate head_pitch base_tilt column_axis_x_bp000">
+      params="parent column base_plate head_pitch base_tilt column_axis_x_bp000 emit_arm_mounts:=true column_inertial:=''">
     <xacro:property name="cfg" lazy_eval="false"
         value="${xacro.load_yaml('$(find openamrobot_upperbody_description)/config/upperbody_configuration.yaml')}"/>
@@ -40,5 +51,13 @@
     <xacro:property name="profile" value="${geo['arm_profile']}" lazy_eval="false"/>
     <!-- Column axis on the base-plate top face (height reference, 304 mm). -->
-    <link name="lift_column_base_link"/>
+    <link name="lift_column_base_link">
+      <xacro:unless value="${column_inertial == ''}">
+        <inertial>
+          <origin xyz="0 0 ${column_inertial['com_z']}" rpy="0 0 0"/>
+          <mass value="${column_inertial['mass']}"/>
+          <inertia ixx="${column_inertial['ixx']}" ixy="0" ixz="0" iyy="${column_inertial['iyy']}" iyz="0" izz="${column_inertial['izz']}"/>
+        </inertial>
+      </xacro:unless>
+    </link>
     <joint name="lift_column_base_joint" type="fixed">
       <parent link="${parent}"/>
@@ -80,6 +99,8 @@
       </joint>
     </xacro:macro>
-    <xacro:openamrobot_arm_mount side="left" sign="1"/>
-    <xacro:openamrobot_arm_mount side="right" sign="-1"/>
+    <xacro:if value="${emit_arm_mounts}">
+      <xacro:openamrobot_arm_mount side="left" sign="1"/>
+      <xacro:openamrobot_arm_mount side="right" sign="-1"/>
+    </xacro:if>
     <!-- Head camera (ZED Mini). head_camera_mount_link is the pitch pivot on the
          lens line; head_camera_link is pitched down by head_pitch about y. -->

Commit message: feat(description): the placeholder boxes get one named material, in the URDF and for Gazebo
lift_column_base_link, lift_carriage_link and arm_profile_link had no <material>: RViz drew them red and Gazebo
black. They now use the material placeholder_geometry (rgba 0.78 0.64 0.45 1.0, a flat cardboard tan nothing
else in the combined robot uses), and each link has a <gazebo reference> block with the same ambient and
diffuse, because sdformat takes a link's colour from that block and a URDF material alone comes out 1.25 times
brighter in the SDF.

sdformat applies that block only to a visual with no name of its own, so the two column visuals lose their
name attribute (their collisions keep placeholder_*). No pose, mount, stop height, frame or joint changes.
test_p25_placeholder_material.py pins the colour in the URDF, the <gazebo> block and the SDF from gz sdf -p;
it fails on the old xacro and on a re-named column visual.

Assisted-by: Claude Code
Signed-off-by: Tushar Goel <Slash8860300674@gmail.com>

File: ros2/src/openamrobot_upperbody_description/urdf/openamrobot_upperbody.xacro (robot description, xacro)
@@ -22,5 +22,5 @@
     column_geometry  '' (none): the column has no visual and no collision. A dict
                      {section_x, section_y}: both stages get a box of that section,
-                     visual and collision, named placeholder_*: the fixed stage on
+                     visual and collision (the collisions named placeholder_*): the fixed stage on
                      lift_column_base_link (retracted length), the moving stage on
                      lift_carriage_link (stroke, below the carriage). Placeholder
@@ -57,4 +57,20 @@
     <xacro:property name="lens" value="${geo['head_camera_lens']}" lazy_eval="false"/>
     <xacro:property name="profile" value="${geo['arm_profile']}" lazy_eval="false"/>
+    <!-- Presentation only, not a datum: one colour for every placeholder box. -->
+    <xacro:property name="placeholder_rgba" value="0.78 0.64 0.45 1.0" lazy_eval="false"/>
+    <material name="placeholder_geometry">
+      <color rgba="${placeholder_rgba}"/>
+    </material>
+    <xacro:macro name="openamrobot_placeholder_gazebo_material" params="link">
+      <gazebo reference="${link}">
+        <visual>
+          <material>
+            <ambient>${placeholder_rgba}</ambient>
+            <diffuse>${placeholder_rgba}</diffuse>
+            <specular>0.1 0.1 0.1 1.0</specular>
+          </material>
+        </visual>
+      </gazebo>
+    </xacro:macro>
     <!-- Column axis on the base-plate top face (height reference, 304 mm). -->
     <link name="lift_column_base_link">
@@ -67,7 +83,8 @@
       </xacro:unless>
       <xacro:unless value="${column_geometry == ''}">
-        <visual name="placeholder_lift_column_fixed_stage">
+        <visual>
           <origin xyz="0 0 ${col['retracted_length'] / 2}" rpy="0 0 0"/>
           <geometry><box size="${column_geometry['section_x']} ${column_geometry['section_y']} ${col['retracted_length']}"/></geometry>
+          <material name="placeholder_geometry"/>
         </visual>
         <collision name="placeholder_lift_column_fixed_stage">
@@ -77,4 +94,7 @@
       </xacro:unless>
     </link>
+    <xacro:unless value="${column_geometry == ''}">
+      <xacro:openamrobot_placeholder_gazebo_material link="lift_column_base_link"/>
+    </xacro:unless>
     <joint name="lift_column_base_joint" type="fixed">
       <parent link="${parent}"/>
@@ -90,7 +110,8 @@
     <xacro:unless value="${column_geometry == ''}">
       <link name="lift_carriage_link">
-        <visual name="placeholder_lift_column_moving_stage">
+        <visual>
           <origin xyz="0 0 ${-col['stroke'] / 2}" rpy="0 0 0"/>
           <geometry><box size="${column_geometry['section_x']} ${column_geometry['section_y']} ${col['stroke']}"/></geometry>
+          <material name="placeholder_geometry"/>
         </visual>
         <collision name="placeholder_lift_column_moving_stage">
@@ -99,4 +120,5 @@
         </collision>
       </link>
+      <xacro:openamrobot_placeholder_gazebo_material link="lift_carriage_link"/>
     </xacro:unless>
     <joint name="lift_joint" type="prismatic">
@@ -111,4 +133,5 @@
       <visual>
         <geometry><box size="${profile['size_x']} ${profile['size_y']} ${profile['length']}"/></geometry>
+        <material name="placeholder_geometry"/>
       </visual>
       <collision>
@@ -116,4 +139,5 @@
       </collision>
     </link>
+    <xacro:openamrobot_placeholder_gazebo_material link="arm_profile_link"/>
     <joint name="arm_profile_joint" type="fixed">
       <parent link="lift_carriage_link"/>
